File: lightball.sch (KiCad schematic (older format))
At the start: 47 parts, among them J1 IN, J2 Conn_01x06, J3 Motor, Q1 2N7002, U1 BMP388, U2 MIC5504-3.3YM5, U3 ACT4088, U4 ESP8266EX, U5 25LCxxx, Y1 Crystal

Commit message: update projects
Parts:
- AE1: footprint Connector_Wire:SolderWirePad_1x01_SMD_5x10mm -> TestPoint:TestPoint_Pad_1.0x1.0mm
Changed lines of the file:
@@
 F 0 "AE1" V 3517 3245 50  0000 C CNN
 F 1 "Antenna" V 3426 3245 50  0000 C CNN
-F 2 "Connector_Wire:SolderWirePad_1x01_SMD_5x10mm" H 3300 3300 50  0001 C CNN
+F 2 "TestPoint:TestPoint_Pad_1.0x1.0mm" H 3300 3300 50  0001 C CNN
 F 3 "~" H 3300 3300 50  0001 C CNN
 	1    3300 3300

Commit message: FIX: better ground connection
Parts:
- removed C16, C17: C_Small, Capacitor_SMD:C_0402_1005Metric, symbol Device:C_Small
- removed Y1: Crystal, stmbl:Crystal_SMD_0603_4Pads, symbol Device:Crystal
- added C18: 1u, Capacitor_SMD:C_0603_1608Metric, symbol Device:C
- added C19: 0.1µ, Capacitor_SMD:C_0402_1005Metric, symbol Device:C
- added Y1: Crystal_GND24, Crystal:Crystal_SMD_SeikoEpson_FA238-4Pin_3.2x2.5mm, symbol Device:Crystal_GND24
- C10, C11, C4, C5: footprint Capacitor_SMD:C_0402_1005Metric -> Capacitor_SMD:C_0603_1608Metric
- C15: value 0.1µ -> 10u
- C7, C9: value 0.1µ -> 10u; footprint Capacitor_SMD:C_0402_1005Metric -> Capacitor_SMD:C_0603_1608Metric
- L2: footprint Inductor_SMD:L_0402_1005Metric -> Inductor_SMD:L_0603_1608Metric
- R5: footprint Resistor_SMD:R_0603_1608Metric -> Resistor_SMD:R_0402_1005Metric
Connections:
- net +3V3: now also C19.1; no longer U4.5 (VDD_RTC)
- net GNDD: now also C18.2, C19.2, Y1.2, Y1.4
- net VPP: now also C18.1
- net at C4.1, U4.27 (XTAL_OUT): now also Y1.1
- net at C5.1, U4.28 (XTAL_IN): now also Y1.3
Changed lines of the file:
@@
-$EndComp
-$Comp
-L Device:Crystal Y1
-U 1 1 5C3F8659
-P 4000 3850
-F 0 "Y1" V 3954 3981 50  0000 L CNN
-F 1 "Crystal" V 4045 3981 50  0000 L CNN
-F 2 "stmbl:Crystal_SMD_0603_4Pads" H 4000 3850 50  0001 C CNN
-F 3 "~" H 4000 3850 50  0001 C CNN
-	1    4000 3850
-	0    1    1    0
 $EndComp
 $Comp
@@
 Wire Wire Line
 	5050 2300 4950 2300
-Connection ~ 5150 2300
-Wire Wire Line
-	5150 2300 5050 2300
-Connection ~ 5250 2300
-Wire Wire Line
-	5250 2300 5150 2300
 Connection ~ 5350 2300
 Wire Wire Line
@@
 F 0 "C5" V 3498 4100 50  0000 C CNN
 F 1 "10p" V 3589 4100 50  0000 C CNN
-F 2 "Capacitor_SMD:C_0402_1005Metric" H 3788 3950 50  0001 C CNN
+F 2 "Capacitor_SMD:C_0603_1608Metric" H 3788 3950 50  0001 C CNN
 F 3 "~" H 3750 4100 50  0001 C CNN
 	1    3750 4100
@@
 F 0 "C4" V 3498 3600 50  0000 C CNN
 F 1 "10p" V 3589 3600 50  0000 C CNN
-F 2 "Capacitor_SMD:C_0402_1005Metric" H 3788 3450 50  0001 C CNN
+F 2 "Capacitor_SMD:C_0603_1608Metric" H 3788 3450 50  0001 C CNN
 F 3 "~" H 3750 3600 50  0001 C CNN
 	1    3750 3600
@@
 P 5650 5850
 F 0 "C9" H 5765 5896 50  0000 L CNN
-F 1 "0.1µ" H 5765 5805 50  0000 L CNN
-F 2 "Capacitor_SMD:C_0402_1005Metric" H 5688 5700 50  0001 C CNN
+F 1 "10u" H 5765 5805 50  0000 L CNN
+F 2 "Capacitor_SMD:C_0603_1608Metric" H 5688 5700 50  0001 C CNN
 F 3 "~" H 5650 5850 50  0001 C CNN
 	1    5650 5850
@@
 F 0 "C10" H 6065 5896 50  0000 L CNN
 F 1 "0.1µ" H 6065 5805 50  0000 L CNN
-F 2 "Capacitor_SMD:C_0402_1005Metric" H 5988 5700 50  0001 C CNN
+F 2 "Capacitor_SMD:C_0603_1608Metric" H 5988 5700 50  0001 C CNN
 F 3 "~" H 5950 5850 50  0001 C CNN
 	1    5950 5850
@@
 F 0 "C11" H 6365 5896 50  0000 L CNN
 F 1 "0.1µ" H 6365 5805 50  0000 L CNN
-F 2 "Capacitor_SMD:C_0402_1005Metric" H 6288 5700 50  0001 C CNN
+F 2 "Capacitor_SMD:C_0603_1608Metric" H 6288 5700 50  0001 C CNN
 F 3 "~" H 6250 5850 50  0001 C CNN
 	1    6250 5850
@@
 P 4300 6900
 F 0 "C7" H 4415 6946 50  0000 L CNN
-F 1 "0.1µ" H 4415 6855 50  0000 L CNN
-F 2 "Capacitor_SMD:C_0402_1005Metric" H 4338 6750 50  0001 C CNN
+F 1 "10u" H 4415 6855 50  0000 L CNN
+F 2 "Capacitor_SMD:C_0603_1608Metric" H 4338 6750 50  0001 C CNN
 F 3 "~" H 4300 6900 50  0001 C CNN
 	1    4300 6900
@@
 F 0 "R5" V 4307 2450 50  0000 C CNN
 F 1 "12k" V 4216 2450 50  0000 C CNN
-F 2 "Resistor_SMD:R_0603_1608Metric" V 4030 2450 50  0001 C CNN
+F 2 "Resistor_SMD:R_0402_1005Metric" V 4030 2450 50  0001 C CNN
 F 3 "~" H 4100 2450 50  0001 C CNN
 	1    4100 2450
@@
 P 8100 6100
 F 0 "C15" H 8215 6146 50  0000 L CNN
-F 1 "0.1µ" H 8215 6055 50  0000 L CNN
+F 1 "10u" H 8215 6055 50  0000 L CNN
 F 2 "Capacitor_SMD:C_0402_1005Metric" H 8138 5950 50  0001 C CNN
 F 3 "~" H 8100 6100 50  0001 C CNN
@@
 	4250 1500 3450 1500
 $Comp
-L Device:C_Small C17
-U 1 1 5BF28D4A
-P 4200 3400
-F 0 "C17" H 4108 3354 50  0000 R CNN
-F 1 "C_Small" H 4108 3445 50  0000 R CNN
-F 2 "Capacitor_SMD:C_0402_1005Metric" H 4200 3400 50  0001 C CNN
-F 3 "~" H 4200 3400 50  0001 C CNN
-	1    4200 3400
-	-1   0    0    1
-$EndComp
-$Comp
-L Device:C_Small C16
-U 1 1 5BF28E92
-P 3900 3400
-F 0 "C16" H 3992 3446 50  0000 L CNN
-F 1 "C_Small" H 3992 3355 50  0000 L CNN
-F 2 "Capacitor_SMD:C_0402_1005Metric" H 3900 3400 50  0001 C CNN
-F 3 "~" H 3900 3400 50  0001 C CNN
-	1    3900 3400
-	1    0    0    -1
-$EndComp
-$Comp
 L Device:L_Small L2
 U 1 1 5BF2916B
@@
 F 0 "L2" V 4235 3300 50  0000 C CNN
 F 1 "L_Small" V 4144 3300 50  0000 C CNN
-F 2 "Inductor_SMD:L_0402_1005Metric" H 4050 3300 50  0001 C CNN
+F 2 "Inductor_SMD:L_0603_1608Metric" H 4050 3300 50  0001 C CNN
 F 3 "~" H 4050 3300 50  0001 C CNN
 	1    4050 3300
 	0    -1   -1   0
 $EndComp
-Wire Wire Line
-	4150 3300 4200 3300
-Connection ~ 4200 3300
-Wire Wire Line
-	4200 3300 4350 3300
-Wire Wire Line
-	3950 3300 3900 3300
-Connection ~ 3900 3300
-Wire Wire Line
-	3900 3300 3500 3300
 $Comp
 L Device:Antenna AE1
@@
 	0    -1   -1   0
 $EndComp
-$Comp
-L power:GNDD #PWR0101
-U 1 1 5BF2D871
-P 3900 3500
-F 0 "#PWR0101" H 3900 3250 50  0001 C CNN
-F 1 "GNDD" V 3904 3390 50  0000 R CNN
-F 2 "" H 3900 3500 50  0001 C CNN
-F 3 "" H 3900 3500 50  0001 C CNN
-	1    3900 3500
+Wire Wire Line
+	5250 2300 5250 2250
+Wire Wire Line
+	5250 2250 5100 2250
+Wire Wire Line
+	5100 2250 5100 2300
+Wire Wire Line
+	5100 2300 5050 2300
+Connection ~ 5250 2300
+$Comp
+L Device:C C18
+U 1 1 5C261FDC
+P 2950 5750
+F 0 "C18" H 3065 5796 50  0000 L CNN
+F 1 "1u" H 3065 5705 50  0000 L CNN
+F 2 "Capacitor_SMD:C_0603_1608Metric" H 2988 5600 50  0001 C CNN
+F 3 "~" H 2950 5750 50  0001 C CNN
+	1    2950 5750
+	1    0    0    -1
+$EndComp
+$Comp
+L power:GNDD #PWR055
+U 1 1 5C2620A0
+P 2950 5900
+F 0 "#PWR055" H 2950 5650 50  0001 C CNN
+F 1 "GNDD" H 2954 5745 50  0000 C CNN
+F 2 "" H 2950 5900 50  0001 C CNN
+F 3 "" H 2950 5900 50  0001 C CNN
+	1    2950 5900
+	1    0    0    -1
+$EndComp
+$Comp
+L power:VPP #PWR054
+U 1 1 5C26210B
+P 2950 5600
+F 0 "#PWR054" H 2950 5450 50  0001 C CNN
+F 1 "VPP" H 2965 5773 50  0000 C CNN
+F 2 "" H 2950 5600 50  0001 C CNN
+F 3 "" H 2950 5600 50  0001 C CNN
+	1    2950 5600
+	1    0    0    -1
+$EndComp
+$Comp
+L Device:Crystal_GND24 Y1
+U 1 1 5C263556
+P 4000 3850
+F 0 "Y1" V 3954 4091 50  0000 L CNN
+F 1 "Crystal_GND24" V 4045 4091 50  0000 L CNN
+F 2 "Crystal:Crystal_SMD_SeikoEpson_FA238-4Pin_3.2x2.5mm" H 4000 3850 50  0001 C CNN
+F 3 "~" H 4000 3850 50  0001 C CNN
+	1    4000 3850
 	0    1    1    0
 $EndComp
 $Comp
-L power:GNDD #PWR0102
-U 1 1 5BF2FCA6
-P 4200 3500
-F 0 "#PWR0102" H 4200 3250 50  0001 C CNN
-F 1 "GNDD" V 4204 3390 50  0000 R CNN
-F 2 "" H 4200 3500 50  0001 C CNN
-F 3 "" H 4200 3500 50  0001 C CNN
-	1    4200 3500
+L power:GNDD #PWR0103
+U 1 1 5C26362D
+P 3800 3850
+F 0 "#PWR0103" H 3800 3600 50  0001 C CNN
+F 1 "GNDD" V 3804 3740 50  0000 R CNN
+F 2 "" H 3800 3850 50  0001 C CNN
+F 3 "" H 3800 3850 50  0001 C CNN
+	1    3800 3850
 	0    1    1    0
 $EndComp
+$Comp
+L power:GNDD #PWR0104
+U 1 1 5C263698
+P 4200 3850
+F 0 "#PWR0104" H 4200 3600 50  0001 C CNN
+F 1 "GNDD" V 4204 3740 50  0000 R CNN
+F 2 "" H 4200 3850 50  0001 C CNN
+F 3 "" H 4200 3850 50  0001 C CNN
+	1    4200 3850
+	0    -1   -1   0
+$EndComp
+$Comp
+L Device:C C19
+U 1 1 5C26591E
+P 3100 6900
+F 0 "C19" H 3215 6946 50  0000 L CNN
+F 1 "0.1µ" H 3215 6855 50  0000 L CNN
+F 2 "Capacitor_SMD:C_0402_1005Metric" H 3138 6750 50  0001 C CNN
+F 3 "~" H 3100 6900 50  0001 C CNN
+	1    3100 6900
+	1    0    0    -1
+$EndComp
+$Comp
+L power:GNDD #PWR057
+U 1 1 5C265925
+P 3100 7050
+F 0 "#PWR057" H 3100 6800 50  0001 C CNN
+F 1 "GNDD" H 3104 6895 50  0000 C CNN
+F 2 "" H 3100 7050 50  0001 C CNN
+F 3 "" H 3100 7050 50  0001 C CNN
+	1    3100 7050
+	1    0    0    -1
+$EndComp
+$Comp
+L power:+3.3V #PWR056
+U 1 1 5C26592B
+P 3100 6750
+F 0 "#PWR056" H 3100 6600 50  0001 C CNN
+F 1 "+3.3V" H 3115 6923 50  0000 C CNN
+F 2 "" H 3100 6750 50  0001 C CNN
+F 3 "" H 3100 6750 50  0001 C CNN
+	1    3100 6750
+	1    0    0    -1
+$EndComp
+Wire Wire Line
+	4150 3300 4350 3300
+Wire Wire Line
+	3500 3300 3950 3300
 $EndSCHEMATC
